Commit message: camera added to robot

File: Day6/tasks/catkin_ws/src/myRobot_description/urdf/model.urdf.xacro (robot description, xacro)
@@ -8,4 +8,5 @@
   <xacro:property name="wheeldiam" value="0.07" />
   <xacro:property name="pi" value="3.1415" />
+  <xacro:property name="camera_link" value="0.05" />
   <material name="blue">
     <color rgba="0 0 0.8 1"/>
@@ -193,8 +194,8 @@
     <origin xyz="0 0 ${bodylen/2}"/>
   </joint>
-  <link name="box">
-    <visual>
-      <geometry>
-        <box size="0.08 0.08 0.08"/>
+  <link name="camera_link">
+    <visual>
+      <geometry>
+        <box size="${camera_link} ${camera_link} ${camera_link}"/>
       </geometry>
       <material name="blue"/>
@@ -203,5 +204,5 @@
     <collision>
       <geometry>
-        <box size="0.08 0.08 0.08"/>
+        <box size="${camera_link} ${camera_link} ${camera_link}"/>
       </geometry>
     </collision>
@@ -210,6 +211,45 @@
   <joint name="tobox" type="fixed">
     <parent link="head"/>
-    <child link="box"/>
+    <child link="camera_link"/>
     <origin xyz="${.707*width+0.04} 0 ${.707*width}"/>
   </joint>
+  <gazebo reference="camera_link">
+    <sensor type="camera" name="camera1">
+      <update_rate>30.0</update_rate>
+      <camera name="camera1">
+        <horizontal_fov>1.3962634</horizontal_fov>
+        <image>
+          <width>800</width>
+          <height>800</height>
+          <format>R8G8B8</format>
+        </image>
+        <clip>
+          <near>0.02</near>
+          <far>300</far>
+        </clip>
+        <noise>
+          <type>gaussian</type>
+          <!-- Noise is sampled independently per pixel on each frame.
+               That pixel's noise value is added to each of its color
+               channels, which at that point lie in the range [0,1]. -->
+          <mean>0.0</mean>
+          <stddev>0.007</stddev>
+        </noise>
+      </camera>
+      <plugin name="camera_controller" filename="libgazebo_ros_camera.so">
+        <alwaysOn>true</alwaysOn>
+        <updateRate>0.0</updateRate>
+        <cameraName>model/camera1</cameraName>
+        <imageTopicName>image_raw</imageTopicName>
+        <cameraInfoTopicName>camera_info</cameraInfoTopicName>
+        <frameName>camera_link</frameName>
+        <hackBaseline>0.07</hackBaseline>
+        <distortionK1>0.0</distortionK1>
+        <distortionK2>0.0</distortionK2>
+        <distortionK3>0.0</distortionK3>
+        <distortionT1>0.0</distortionT1>
+        <distortionT2>0.0</distortionT2>
+      </plugin>
+    </sensor>
+  </gazebo>
 </robot>

Commit message: laser added

File: Day6/tasks/catkin_ws/src/myRobot_description/urdf/model.urdf.xacro (robot description, xacro)
@@ -108,70 +108,64 @@
   <xacro:leg prefix="right" reflect="-1" />
   <xacro:leg prefix="left" reflect="1" />
-  <joint name="gripper_extension" type="prismatic">
+  <joint name="hokuyo_joint" type="fixed">
+    <axis xyz="0 0 0"/>
+     <origin rpy="0 0 0" xyz="${width-.01} 0 0.2"/>
     <parent link="base_link"/>
-    <child link="gripper_pole"/>
-    <limit effort="1000.0" lower="-${width*2-.02}" upper="0" velocity="0.5"/>
-    <origin rpy="0 0 0" xyz="${width-.01} 0 0.2"/>
+    <child link="hokuyo_link"/>
   </joint>
-  <link name="gripper_pole">
-    <visual>
-      <geometry>
-        <cylinder length="${polelen}" radius="0.01"/>
-      </geometry>
+  <link name="hokuyo_link">
+    <collision>
       <origin xyz="${polelen/2} 0 0" rpy="0 ${pi/2} 0 "/>
-    </visual>
-    <collision>
-      <geometry>
-        <cylinder length="${polelen}" radius="0.01"/>
-      </geometry>
-      <origin xyz="${polelen/2} 0 0" rpy="0 ${pi/2} 0 "/>
-    </collision>
-    <xacro:default_inertial mass="0.05"/>
-  </link>
-  <xacro:macro name="gripper" params="prefix reflect">
-    <joint name="${prefix}_gripper_joint" type="revolute">
-      <axis xyz="0 0 ${reflect}"/>
-      <limit effort="1000.0" lower="0.0" upper="0.548" velocity="0.5"/>
-      <origin rpy="0 0 0" xyz="${polelen} ${reflect*0.01} 0"/>
-      <parent link="gripper_pole"/>
-      <child link="${prefix}_gripper"/>
-    </joint>
-    <link name="${prefix}_gripper">
-      <visual>
-        <origin rpy="${(reflect-1)/2*pi} 0 0" xyz="0 0 0"/>
-        <geometry>
-          <mesh filename="package://myRobot_description/meshes/l_finger.dae"/>
-        </geometry>
-      </visual>
-      <collision>
-        <geometry>
-          <mesh filename="package://myRobot_description/meshes/l_finger.dae"/>
-        </geometry>
-        <origin rpy="${(reflect-1)/2*pi} 0 0" xyz="0 0 0"/>
-      </collision>
-      <xacro:default_inertial mass="0.05"/>
-    </link>
-    <joint name="${prefix}_tip_joint" type="fixed">
-      <parent link="${prefix}_gripper"/>
-      <child link="${prefix}_tip"/>
-    </joint>
-    <link name="${prefix}_tip">
-      <visual>
-        <origin rpy="${(reflect-1)/2*pi} 0 0" xyz="0.09137 0.00495 0"/>
-        <geometry>
-          <mesh filename="package://myRobot_description/meshes/l_finger_tip.dae"/>
-        </geometry>
-      </visual>
-      <collision>
-        <geometry>
-          <mesh filename="package://myRobot_description/meshes/l_finger_tip.dae"/>
-        </geometry>
-        <origin rpy="${(reflect-1)/2*pi} 0 0" xyz="0.09137 0.00495 0"/>
-      </collision>
-      <xacro:default_inertial mass="0.05"/>
-    </link>
-  </xacro:macro>
-  <xacro:gripper prefix="left" reflect="1" />
-  <xacro:gripper prefix="right" reflect="-1" />
+      <geometry>
+    <box size="0.1 0.1 0.1"/>
+      </geometry>
+    </collision>
+    <visual>
+     <origin xyz="${polelen/2} 0 0" rpy="0 ${pi/2} 0 "/>
+      <geometry>
+        <mesh filename="package://myRobot_description/meshes/hokuyo.dae"/>
+      </geometry>
+    </visual>
+   <inertial>
+      <mass value="1e-5" />
+      <origin xyz="0 0 0" rpy="0 0 0"/>
+      <inertia ixx="1e-6" ixy="0" ixz="0" iyy="1e-6" iyz="0" izz="1e-6" />
+    </inertial>
+  </link>
+<gazebo reference="hokuyo_link">
+    <sensor type="gpu_ray" name="head_hokuyo_sensor">
+      <pose>0 0 0 0 0 0</pose>
+      <visualize>true</visualize>
+      <update_rate>40</update_rate>
+      <ray>
+        <scan>
+          <horizontal>
+            <samples>720</samples>
+            <resolution>1</resolution>
+            <min_angle>-1.570796</min_angle>
+            <max_angle>1.570796</max_angle>
+          </horizontal>
+        </scan>
+        <range>
+          <min>0.10</min>
+          <max>30.0</max>
+          <resolution>0.01</resolution>
+        </range>
+        <noise>
+          <type>gaussian</type>
+          <!-- Noise parameters based on published spec for Hokuyo laser
+               achieving "+-30mm" accuracy at range < 10m.  A mean of 0.0m and
+               stddev of 0.01m will put 99.7% of samples within 0.03m of the true
+               reading. -->
+          <mean>0.0</mean>
+          <stddev>0.01</stddev>
+        </noise>
+      </ray>
+      <plugin name="gazebo_ros_head_hokuyo_controller" filename="libgazebo_ros_gpu_laser.so">
+        <topicName>/model/laser/scan</topicName>
+        <frameName>hokuyo_link</frameName>
+      </plugin>
+    </sensor>
+  </gazebo>
   <link name="head">
     <visual>
